Commit message: Edited URDF to start the robot on the table with fingers

File: robots/common/franka_arm.xacro (robot description, xacro)
@@ -21,6 +21,6 @@
     </xacro:if>
     <xacro:unless value="${not connected_to}">
-      <link name="${connected_to}">
-      </link>
+      <!-- <link name="${connected_to}">
+      </link> -->
       <joint name="${prefix}${connected_to}_joint" type="fixed">
         <parent link="${connected_to}"/>

File: robots/common/franka_robot.xacro (robot description, xacro)
@@ -16,4 +16,9 @@
                       gazebo:='false'
                       with_sc:='false'
+                      ros2_control:=false
+                      robot_ip:=''
+                      use_fake_hardware:=false
+                      fake_sensor_commands:=false
+                      gazebo_effort:=false
                       no_prefix:='false'
                       arm_prefix:=''
@@ -141,4 +146,17 @@
       </xacro:if>
     </xacro:if>
+    <xacro:if value="${ros2_control}">
+      <xacro:include filename="$(find franka_description)/robots/common/franka_arm.ros2_control.xacro"/>
+      <xacro:franka_arm_ros2_control
+          arm_id="${robot_type}"
+          robot_ip="${robot_ip}"
+          use_fake_hardware="${use_fake_hardware}"
+          fake_sensor_commands="${fake_sensor_commands}"
+          gazebo="${gazebo}"
+          hand="${hand}"
+          gazebo_effort="${gazebo_effort}"
+          arm_prefix="${arm_prefix}"
+      />
+    </xacro:if>
   </xacro:macro>
 </robot>

Commit message: dual arm setup:
- add arm_id to hardware interface component name
- add mesh_model as prefix for .dae/.stl files

File: robots/common/franka_arm.xacro (robot description, xacro)
@@ -8,5 +8,5 @@
   <!-- inertials: description of the inertials that comes from a YAML file. Example definition: ${xacro.load_yaml('$(find franka_description)/robots/fr3/inertials.yaml')} -->
   <!-- dynamics: description of the dynamics that comes from a YAML file. Example definition: ${xacro.load_yaml('$(find franka_description)/robots/fr3/dynamics.yaml')} -->
-  <xacro:macro name="franka_arm" params="robot_type arm_prefix:='' no_prefix:=false description_pkg:='franka_description' connected_to:='base' xyz:='0 0 0' rpy:='0 0 0' gazebo:='false' safety_distance:=0 with_sc:=false" >
+  <xacro:macro name="franka_arm" params="robot_type arm_prefix:='' no_prefix:=false description_pkg:='franka_description' connected_to:='base' xyz:='0 0 0' rpy:='0 0 0' gazebo:='false' safety_distance:=0 with_sc:=false mesh_model:=''" >
     <xacro:property name="joint_limits" value="${xacro.load_yaml('$(find franka_description)/robots/' + robot_type + '/joint_limits.yaml')}"/>
     <xacro:property name="inertials" value="${xacro.load_yaml('$(find franka_description)/robots/' + robot_type  + '/inertials.yaml')}"/>
@@ -29,10 +29,10 @@
       </joint>
     </xacro:unless>
-    <xacro:link_with_sc no_prefix="${no_prefix}" name="link0" gazebo="${gazebo}" with_sc="${with_sc}" with_accelerometers="${with_accelerometers}">
+    <xacro:link_with_sc no_prefix="${no_prefix}" name="link0" gazebo="${gazebo}" with_sc="${with_sc}" with_accelerometers="${with_accelerometers}" mesh_model="${mesh_model}">
       <self_collision_geometries>
         <xacro:collision_capsule xyz="-0.075 0 0.06" direction="x" radius="${0.06+safety_distance}" length="0.03" />
       </self_collision_geometries>
     </xacro:link_with_sc>
-    <xacro:link_with_sc no_prefix="${no_prefix}" name="link1" gazebo="${gazebo}" with_sc="${with_sc}" with_accelerometers="${with_accelerometers}">
+    <xacro:link_with_sc no_prefix="${no_prefix}" name="link1" gazebo="${gazebo}" with_sc="${with_sc}" with_accelerometers="${with_accelerometers}" mesh_model="${mesh_model}">
       <self_collision_geometries>
         <xacro:collision_capsule xyz="0 0 -191.5e-3" radius="${0.06+safety_distance}" length="0.283" />
@@ -47,5 +47,5 @@
       <xacro:franka-dynamics name="joint1" config="${dynamics}" />
     </joint>
-    <xacro:link_with_sc no_prefix="${no_prefix}" name="link2" gazebo="${gazebo}" with_sc="${with_sc}" with_accelerometers="${with_accelerometers}">
+    <xacro:link_with_sc no_prefix="${no_prefix}" name="link2" gazebo="${gazebo}" with_sc="${with_sc}" with_accelerometers="${with_accelerometers}" mesh_model="${mesh_model}">
       <self_collision_geometries>
         <xacro:collision_capsule xyz="0 0 0" radius="${0.06+safety_distance}" length="0.12" />
@@ -60,5 +60,5 @@
       <xacro:franka-dynamics name="joint2" config="${dynamics}" />
     </joint>
-    <xacro:link_with_sc no_prefix="${no_prefix}" name="link3" gazebo="${gazebo}" with_sc="${with_sc}" with_accelerometers="${with_accelerometers}">
+    <xacro:link_with_sc no_prefix="${no_prefix}" name="link3" gazebo="${gazebo}" with_sc="${with_sc}" with_accelerometers="${with_accelerometers}" mesh_model="${mesh_model}">
       <self_collision_geometries>
         <xacro:collision_capsule xyz="0 0 -0.145" radius="${0.06+safety_distance}" length="0.15" />
@@ -73,5 +73,5 @@
       <xacro:franka-dynamics name="joint3" config="${dynamics}" />
     </joint>
-    <xacro:link_with_sc no_prefix="${no_prefix}" name="link4" gazebo="${gazebo}" with_sc="${with_sc}" with_accelerometers="${with_accelerometers}">
+    <xacro:link_with_sc no_prefix="${no_prefix}" name="link4" gazebo="${gazebo}" with_sc="${with_sc}" with_accelerometers="${with_accelerometers}" mesh_model="${mesh_model}">
       <self_collision_geometries>
         <xacro:collision_capsule xyz="0 0 0" radius="${0.06+safety_distance}" length="0.12" />
@@ -86,5 +86,5 @@
       <xacro:franka-dynamics name="joint4" config="${dynamics}" />
     </joint>
-    <xacro:link_with_sc no_prefix="${no_prefix}" name="link5" gazebo="${gazebo}" with_sc="${with_sc}" with_accelerometers="${with_accelerometers}">
+    <xacro:link_with_sc no_prefix="${no_prefix}" name="link5" gazebo="${gazebo}" with_sc="${with_sc}" with_accelerometers="${with_accelerometers}" mesh_model="${mesh_model}">
       <self_collision_geometries>
         <xacro:collision_capsule xyz="0 0 -0.26"    radius="${0.060+safety_distance}" length="0.10" />
@@ -100,5 +100,5 @@
       <xacro:franka-dynamics name="joint5" config="${dynamics}" />
     </joint>
-    <xacro:link_with_sc no_prefix="${no_prefix}" name="link6" gazebo="${gazebo}" with_sc="${with_sc}" with_accelerometers="false">
+    <xacro:link_with_sc no_prefix="${no_prefix}" name="link6" gazebo="${gazebo}" with_sc="${with_sc}" with_accelerometers="false" mesh_model="${mesh_model}">
       <self_collision_geometries>
         <xacro:collision_capsule xyz="0 0 -0.03" radius="${0.05+safety_distance}" length="0.08" />
@@ -113,5 +113,5 @@
       <xacro:franka-dynamics name="joint6" config="${dynamics}" />
     </joint>
-    <xacro:link_with_sc no_prefix="${no_prefix}" name="link7" gazebo="${gazebo}" rpy="0 0 ${pi/4}" with_sc="${with_sc}" with_accelerometers="false">
+    <xacro:link_with_sc no_prefix="${no_prefix}" name="link7" gazebo="${gazebo}" rpy="0 0 ${pi/4}" with_sc="${with_sc}" with_accelerometers="false" mesh_model="${mesh_model}">
       <self_collision_geometries>
         <xacro:collision_capsule xyz="0 0 0.01" direction="z" radius="${0.04+safety_distance}" length="0.14" />

File: robots/common/franka_robot.xacro (robot description, xacro)
@@ -25,5 +25,6 @@
                       description_pkg:='franka_description'
                       connected_to:='base'
-                      scheduling_policy:='detached'">
+                      scheduling_policy:='detached'
+                      mesh_model:=''">
     <xacro:include filename="$(find franka_description)/robots/common/utils.xacro" />
     <xacro:include filename="$(find franka_description)/robots/common/franka_arm.xacro"/>
@@ -38,4 +39,5 @@
       with_sc="${with_sc}"
       connected_to="${connected_to}"
+      mesh_model="${mesh_model}"
     />
     <xacro:if value="${hand and ee_id== 'franka_hand'}">

File: robots/common/utils.xacro (robot description, xacro)
@@ -32,16 +32,17 @@
   <!-- self_collision_geometries:  self <collision> models        -->
   <!-- ========================================================== -->
-  <xacro:macro name="link_with_sc" params="name no_prefix:='false' rpy:='0 0 0' **self_collision_geometries gazebo:=false with_sc:=false with_accelerometers:=false">
+  <xacro:macro name="link_with_sc" params="name no_prefix:='false' rpy:='0 0 0' **self_collision_geometries gazebo:=false with_sc:=false with_accelerometers:=false mesh_model:=''">
     <xacro:property name="prefix" value="${'' if no_prefix else arm_prefix + robot_type + '_'}" />
+    <xacro:property name="mesh_id" value="${mesh_model if mesh_model else robot_type}" />
     <!-- sub-link defining detailed meshes for collision with environment -->
     <link name="${prefix}${name}">
       <visual name="${prefix}${name}_visual">
         <geometry>
-          <mesh filename="package://${description_pkg}/meshes/robots/${robot_type}/visual/${name}.dae" />
+          <mesh filename="package://${description_pkg}/meshes/robots/${mesh_id}/visual/${name}.dae" />
         </geometry>
       </visual>
       <collision name="${prefix}${name}_collision">
         <geometry>
-          <mesh filename="package://franka_description/meshes/robots/${robot_type}/collision/${name}.stl" />
+          <mesh filename="package://franka_description/meshes/robots/${mesh_id}/collision/${name}.stl" />
         </geometry>
       </collision>
