Commit message: Edited URDF to start the robot on the table with fingers

File: robots/common/franka_arm.ros2_control.xacro (robot description, xacro)
@@ -15,5 +15,5 @@
         <xacro:if value="${is_async}">
           <properties>
-            <async scheduling_policy="detached" print_warnings="true" thread_priority="${thread_priority}" manage_overruns="false"/>
+            <async scheduling_policy="slave" print_warnings="true" thread_priority="${thread_priority}" manage_overruns="false"/>
           </properties>
         </xacro:if>

File: robots/common/franka_arm.xacro (robot description, xacro)
@@ -16,6 +16,6 @@
     </xacro:if>
     <xacro:unless value="${not connected_to}">
-      <link name="${connected_to}">
-      </link>
+      <!-- <link name="${connected_to}">
+      </link> -->
       <joint name="${prefix}${connected_to}_joint" type="fixed">
         <parent link="${connected_to}"/>

Commit message: Edited URDF to start the robot on the table with fingers

File: robots/common/franka_arm.ros2_control.xacro (robot description, xacro)
@@ -17,5 +17,5 @@
           <param name="prefix">${arm_prefix}</param>
           <xacro:if value="${use_fake_hardware}">
-            <plugin>fake_components/GenericSystem</plugin>
+            <plugin>mock_components/GenericSystem</plugin>
             <param name="fake_sensor_commands">${fake_sensor_commands}</param>
             <param name="state_following_offset">0.0</param>
@@ -58,5 +58,5 @@
       <xacro:configure_joint joint_name="${arm_prefix}${arm_id}_joint6" initial_position="${pi/2}"/>
       <xacro:configure_joint joint_name="${arm_prefix}${arm_id}_joint7" initial_position="${pi/4}"/>
-      <xacro:if value="${gazebo and hand}">
+      <xacro:if value="${hand}">
         <xacro:configure_joint joint_name="${arm_prefix}${arm_id}_finger_joint1" initial_position="0.0" />
       </xacro:if>

File: robots/common/franka_arm.xacro (robot description, xacro)
@@ -2,10 +2,4 @@
 <robot xmlns:xacro="http://www.ros.org/wiki/xacro" name="franka_arm">
   <xacro:include filename="$(find franka_description)/robots/common/utils.xacro" />
-  <!-- safety_distance: Minimum safety distance in [m] by which the collision volumes are expanded and which is enforced during robot motions -->
-  <!-- arm_id: Namespace of the robot arm. Serves to differentiate between arms in case of multiple instances. -->
-  <!-- joint_limits: description of the joint limits that comes from a YAML file. Example definition: ${xacro.load_yaml('$(find franka_description)/robots/fr3/joint_limits.yaml')} -->
-  <!-- kinematics: description of the kinematics that comes from a YAML file. Example definition: ${xacro.load_yaml('$(find franka_description)/robots/fr3/kinematics.yaml')} -->
-  <!-- inertials: description of the inertials that comes from a YAML file. Example definition: ${xacro.load_yaml('$(find franka_description)/robots/fr3/inertials.yaml')} -->
-  <!-- dynamics: description of the dynamics that comes from a YAML file. Example definition: ${xacro.load_yaml('$(find franka_description)/robots/fr3/dynamics.yaml')} -->
   <xacro:macro name="franka_arm" params="arm_id arm_prefix:='' no_prefix:=false description_pkg:='franka_description' connected_to:='base' xyz:='0 0 0' rpy:='0 0 0' gazebo:='false' safety_distance:=0 joint_limits inertials kinematics dynamics with_sc:=false" >
     <!-- Define a property that defaults to 'arm_prefix_arm_id' concatenated with an underscore if 'no_prefix' is not set -->
@@ -15,6 +9,6 @@
     </xacro:if>
     <xacro:unless value="${not connected_to}">
-      <link name="${connected_to}">
-      </link>
+      <!-- <link name="${connected_to}">
+      </link> -->
       <joint name="${prefix}${connected_to}_joint" type="fixed">
         <parent link="${connected_to}"/>

Commit message: add slave mode async hw for fr3 ros2_control

File: robots/common/franka_arm.ros2_control.xacro (robot description, xacro)
@@ -12,10 +12,9 @@
                  is_async:=false
                  thread_priority:=50">
-    <ros2_control name="${arm_prefix}FrankaHardwareInterface" type="system" is_async="${is_async}">
-        <xacro:if value="${is_async}">
-          <properties>
-            <async scheduling_policy="slave" print_warnings="true" thread_priority="${thread_priority}" manage_overruns="false"/>
-          </properties>
-        </xacro:if>
+    <xacro:property name="arm_prefix_modified" value="${'' if arm_prefix == '' else arm_prefix + '_'}" />
+    <ros2_control name="${arm_prefix_modified}FrankaHardwareInterface" type="system" is_async="true" rw_rate="1000">
+        <properties>
+            <async scheduling_policy="slave" print_warnings="true" thread_priority="${thread_priority}"/>
+        </properties>
         <hardware>
           <param name="version">1.0.0</param>

Commit message: dual arm setup:
- add arm_id to hardware interface component name
- add mesh_model as prefix for .dae/.stl files

File: robots/common/franka_arm.ros2_control.xacro (robot description, xacro)
@@ -76,14 +76,14 @@
       </xacro:macro>
       <!-- Cartesian velocity interfaces -->
-      <xacro:general_purpose_io prefix="vx" command_interface="cartesian_velocity" index="0"/>
-      <xacro:general_purpose_io prefix="vy" command_interface="cartesian_velocity" index="1"/>
-      <xacro:general_purpose_io prefix="vz" command_interface="cartesian_velocity" index="2"/>
-      <xacro:general_purpose_io prefix="wx" command_interface="cartesian_velocity" index="3"/>
-      <xacro:general_purpose_io prefix="wy" command_interface="cartesian_velocity" index="4"/>
-      <xacro:general_purpose_io prefix="wz" command_interface="cartesian_velocity" index="5"/>
+      <xacro:general_purpose_io prefix="${arm_prefix}${arm_id}_vx" command_interface="cartesian_velocity" index="0"/>
+      <xacro:general_purpose_io prefix="${arm_prefix}${arm_id}_vy" command_interface="cartesian_velocity" index="1"/>
+      <xacro:general_purpose_io prefix="${arm_prefix}${arm_id}_vz" command_interface="cartesian_velocity" index="2"/>
+      <xacro:general_purpose_io prefix="${arm_prefix}${arm_id}_wx" command_interface="cartesian_velocity" index="3"/>
+      <xacro:general_purpose_io prefix="${arm_prefix}${arm_id}_wy" command_interface="cartesian_velocity" index="4"/>
+      <xacro:general_purpose_io prefix="${arm_prefix}${arm_id}_wz" command_interface="cartesian_velocity" index="5"/>
       <!-- Cartesian pose interfaces, in total 16 interfaces -->
       <xacro:macro name="loop" params="i">
         <xacro:unless value="${i == 16}">
-          <xacro:general_purpose_io prefix="${i}" command_interface="cartesian_pose_command" index="${i}"/>
+          <xacro:general_purpose_io prefix="${arm_prefix}${arm_id}_${i}" command_interface="cartesian_pose_command" index="${i}"/>
           <xacro:loop i="${i+1}"/>
         </xacro:unless>
@@ -91,6 +91,6 @@
       <xacro:loop i="0"/>
       <!-- Elbow command interfaces -->
-      <xacro:general_purpose_io prefix="joint_3_position" command_interface="elbow_command" index="0"/>
-      <xacro:general_purpose_io prefix="joint_4_sign" command_interface="elbow_command" index="1"/>
+      <xacro:general_purpose_io prefix="${arm_prefix}${arm_id}_joint_3_position" command_interface="elbow_command" index="0"/>
+      <xacro:general_purpose_io prefix="${arm_prefix}${arm_id}_joint_4_sign" command_interface="elbow_command" index="1"/>
     </ros2_control>
     <xacro:if value="${gazebo}">

File: robots/common/franka_arm.xacro (robot description, xacro)
@@ -8,5 +8,5 @@
   <!-- inertials: description of the inertials that comes from a YAML file. Example definition: ${xacro.load_yaml('$(find franka_description)/robots/fr3/inertials.yaml')} -->
   <!-- dynamics: description of the dynamics that comes from a YAML file. Example definition: ${xacro.load_yaml('$(find franka_description)/robots/fr3/dynamics.yaml')} -->
-  <xacro:macro name="franka_arm" params="robot_type arm_prefix:='' no_prefix:=false description_pkg:='franka_description' connected_to:='base' xyz:='0 0 0' rpy:='0 0 0' gazebo:='false' safety_distance:=0 joint_limits inertials kinematics accelerometer_config dynamics with_sc:=false" >
+  <xacro:macro name="franka_arm" params="robot_type arm_prefix:='' no_prefix:=false description_pkg:='franka_description' connected_to:='base' xyz:='0 0 0' rpy:='0 0 0' gazebo:='false' safety_distance:=0 joint_limits inertials kinematics accelerometer_config dynamics with_sc:=false mesh_model:=''" >
     <!-- Define a property that defaults to 'arm_prefix_robot_type' concatenated with an underscore if 'no_prefix' is not set -->
     <xacro:property name="prefix" value="${'' if no_prefix else arm_prefix + robot_type + '_'}" />
@@ -24,10 +24,10 @@
       </joint>
     </xacro:unless>
-    <xacro:link_with_sc no_prefix="${no_prefix}" name="link0" gazebo="${gazebo}" with_sc="${with_sc}" with_accelerometers="${with_accelerometers}">
+    <xacro:link_with_sc no_prefix="${no_prefix}" name="link0" gazebo="${gazebo}" with_sc="${with_sc}" with_accelerometers="${with_accelerometers}" mesh_model="${mesh_model}">
       <self_collision_geometries>
         <xacro:collision_capsule xyz="-0.075 0 0.06" direction="x" radius="${0.06+safety_distance}" length="0.03" />
       </self_collision_geometries>
     </xacro:link_with_sc>
-    <xacro:link_with_sc no_prefix="${no_prefix}" name="link1" gazebo="${gazebo}" with_sc="${with_sc}" with_accelerometers="${with_accelerometers}">
+    <xacro:link_with_sc no_prefix="${no_prefix}" name="link1" gazebo="${gazebo}" with_sc="${with_sc}" with_accelerometers="${with_accelerometers}" mesh_model="${mesh_model}">
       <self_collision_geometries>
         <xacro:collision_capsule xyz="0 0 -191.5e-3" radius="${0.06+safety_distance}" length="0.283" />
@@ -42,5 +42,5 @@
       <xacro:franka-dynamics name="joint1" config="${dynamics}" />
     </joint>
-    <xacro:link_with_sc no_prefix="${no_prefix}" name="link2" gazebo="${gazebo}" with_sc="${with_sc}" with_accelerometers="${with_accelerometers}">
+    <xacro:link_with_sc no_prefix="${no_prefix}" name="link2" gazebo="${gazebo}" with_sc="${with_sc}" with_accelerometers="${with_accelerometers}" mesh_model="${mesh_model}">
       <self_collision_geometries>
         <xacro:collision_capsule xyz="0 0 0" radius="${0.06+safety_distance}" length="0.12" />
@@ -55,5 +55,5 @@
       <xacro:franka-dynamics name="joint2" config="${dynamics}" />
     </joint>
-    <xacro:link_with_sc no_prefix="${no_prefix}" name="link3" gazebo="${gazebo}" with_sc="${with_sc}" with_accelerometers="${with_accelerometers}">
+    <xacro:link_with_sc no_prefix="${no_prefix}" name="link3" gazebo="${gazebo}" with_sc="${with_sc}" with_accelerometers="${with_accelerometers}" mesh_model="${mesh_model}">
       <self_collision_geometries>
         <xacro:collision_capsule xyz="0 0 -0.145" radius="${0.06+safety_distance}" length="0.15" />
@@ -68,5 +68,5 @@
       <xacro:franka-dynamics name="joint3" config="${dynamics}" />
     </joint>
-    <xacro:link_with_sc no_prefix="${no_prefix}" name="link4" gazebo="${gazebo}" with_sc="${with_sc}" with_accelerometers="${with_accelerometers}">
+    <xacro:link_with_sc no_prefix="${no_prefix}" name="link4" gazebo="${gazebo}" with_sc="${with_sc}" with_accelerometers="${with_accelerometers}" mesh_model="${mesh_model}">
       <self_collision_geometries>
         <xacro:collision_capsule xyz="0 0 0" radius="${0.06+safety_distance}" length="0.12" />
@@ -81,5 +81,5 @@
       <xacro:franka-dynamics name="joint4" config="${dynamics}" />
     </joint>
-    <xacro:link_with_sc no_prefix="${no_prefix}" name="link5" gazebo="${gazebo}" with_sc="${with_sc}" with_accelerometers="${with_accelerometers}">
+    <xacro:link_with_sc no_prefix="${no_prefix}" name="link5" gazebo="${gazebo}" with_sc="${with_sc}" with_accelerometers="${with_accelerometers}" mesh_model="${mesh_model}">
       <self_collision_geometries>
         <xacro:collision_capsule xyz="0 0 -0.26"    radius="${0.060+safety_distance}" length="0.10" />
@@ -95,5 +95,5 @@
       <xacro:franka-dynamics name="joint5" config="${dynamics}" />
     </joint>
-    <xacro:link_with_sc no_prefix="${no_prefix}" name="link6" gazebo="${gazebo}" with_sc="${with_sc}" with_accelerometers="false">
+    <xacro:link_with_sc no_prefix="${no_prefix}" name="link6" gazebo="${gazebo}" with_sc="${with_sc}" with_accelerometers="false" mesh_model="${mesh_model}">
       <self_collision_geometries>
         <xacro:collision_capsule xyz="0 0 -0.03" radius="${0.05+safety_distance}" length="0.08" />
@@ -108,5 +108,5 @@
       <xacro:franka-dynamics name="joint6" config="${dynamics}" />
     </joint>
-    <xacro:link_with_sc no_prefix="${no_prefix}" name="link7" gazebo="${gazebo}" rpy="0 0 ${pi/4}" with_sc="${with_sc}" with_accelerometers="false">
+    <xacro:link_with_sc no_prefix="${no_prefix}" name="link7" gazebo="${gazebo}" rpy="0 0 ${pi/4}" with_sc="${with_sc}" with_accelerometers="false" mesh_model="${mesh_model}">
       <self_collision_geometries>
         <xacro:collision_capsule xyz="0 0 0.01" direction="z" radius="${0.04+safety_distance}" length="0.14" />

File: robots/common/franka_robot.xacro (robot description, xacro)
@@ -32,5 +32,6 @@
                       is_async:=false
                       thread_priority:=50
-                      scheduling_policy:='detached'">
+                      scheduling_policy:='detached'
+                      mesh_model:=''">
     <xacro:include filename="$(find franka_description)/robots/common/utils.xacro" />
     <xacro:include filename="$(find franka_description)/robots/common/franka_arm.xacro"/>
@@ -50,4 +51,5 @@
       with_sc="${with_sc}"
       connected_to="${connected_to}"
+      mesh_model="${mesh_model}"
     />
     <xacro:if value="${hand and ee_id == 'franka_hand'}">
