Commit message: dual arm setup:
- add arm_id to hardware interface component name
- add mesh_model as prefix for .dae/.stl files

File: robots/common/franka_arm.ros2_control.xacro (robot description, xacro)
@@ -12,5 +12,5 @@
                  scheduling_policy:=detached">
     <xacro:property name="arm_prefix_modified" value="${'' if arm_prefix == '' else arm_prefix + '_'}" />
-    <ros2_control name="${arm_prefix_modified}FrankaHardwareInterface" type="system" is_async="${use_fake_hardware == 0}" rw_rate="1000">
+    <ros2_control name="${arm_prefix_modified}${arm_id}_FrankaHardwareInterface" type="system" is_async="${use_fake_hardware == 0}" rw_rate="1000">
         <xacro:if value="${use_fake_hardware == 0 and gazebo == 0}">
             <properties>
@@ -74,14 +74,14 @@
       </xacro:macro>
       <!-- Cartesian velocity interfaces -->
-      <xacro:general_purpose_io prefix="vx" command_interface="cartesian_velocity" index="0"/>
-      <xacro:general_purpose_io prefix="vy" command_interface="cartesian_velocity" index="1"/>
-      <xacro:general_purpose_io prefix="vz" command_interface="cartesian_velocity" index="2"/>
-      <xacro:general_purpose_io prefix="wx" command_interface="cartesian_velocity" index="3"/>
-      <xacro:general_purpose_io prefix="wy" command_interface="cartesian_velocity" index="4"/>
-      <xacro:general_purpose_io prefix="wz" command_interface="cartesian_velocity" index="5"/>
+      <xacro:general_purpose_io prefix="${arm_prefix}${arm_id}_vx" command_interface="cartesian_velocity" index="0"/>
+      <xacro:general_purpose_io prefix="${arm_prefix}${arm_id}_vy" command_interface="cartesian_velocity" index="1"/>
+      <xacro:general_purpose_io prefix="${arm_prefix}${arm_id}_vz" command_interface="cartesian_velocity" index="2"/>
+      <xacro:general_purpose_io prefix="${arm_prefix}${arm_id}_wx" command_interface="cartesian_velocity" index="3"/>
+      <xacro:general_purpose_io prefix="${arm_prefix}${arm_id}_wy" command_interface="cartesian_velocity" index="4"/>
+      <xacro:general_purpose_io prefix="${arm_prefix}${arm_id}_wz" command_interface="cartesian_velocity" index="5"/>
       <!-- Cartesian pose interfaces, in total 16 interfaces -->
       <xacro:macro name="loop" params="i">
         <xacro:unless value="${i == 16}">
-          <xacro:general_purpose_io prefix="${i}" command_interface="cartesian_pose_command" index="${i}"/>
+          <xacro:general_purpose_io prefix="${arm_prefix}${arm_id}_${i}" command_interface="cartesian_pose_command" index="${i}"/>
           <xacro:loop i="${i+1}"/>
         </xacro:unless>
@@ -89,6 +89,6 @@
       <xacro:loop i="0"/>
       <!-- Elbow command interfaces -->
-      <xacro:general_purpose_io prefix="joint_3_position" command_interface="elbow_command" index="0"/>
-      <xacro:general_purpose_io prefix="joint_4_sign" command_interface="elbow_command" index="1"/>
+      <xacro:general_purpose_io prefix="${arm_prefix}${arm_id}_joint_3_position" command_interface="elbow_command" index="0"/>
+      <xacro:general_purpose_io prefix="${arm_prefix}${arm_id}_joint_4_sign" command_interface="elbow_command" index="1"/>
     </ros2_control>
     <xacro:if value="${gazebo}">

File: robots/common/franka_arm.xacro (robot description, xacro)
@@ -2,5 +2,5 @@
 <robot xmlns:xacro="http://www.ros.org/wiki/xacro" name="franka_arm">
   <xacro:include filename="$(find franka_description)/robots/common/utils.xacro" />
-  <xacro:macro name="franka_arm" params="arm_id arm_prefix:='' no_prefix:=false description_pkg:='franka_description' connected_to:='base' xyz:='0 0 0' rpy:='0 0 0' gazebo:='false' safety_distance:=0 joint_limits inertials kinematics dynamics with_sc:=false" >
+  <xacro:macro name="franka_arm" params="arm_id arm_prefix:='' no_prefix:=false description_pkg:='franka_description' connected_to:='base' xyz:='0 0 0' rpy:='0 0 0' gazebo:='false' safety_distance:=0 joint_limits inertials kinematics dynamics with_sc:=false mesh_model:=''" >
     <!-- Define a property that defaults to 'arm_prefix_arm_id' concatenated with an underscore if 'no_prefix' is not set -->
     <xacro:property name="prefix" value="${'' if no_prefix else arm_prefix + arm_id + '_'}" />
@@ -17,10 +17,10 @@
       </joint>
     </xacro:unless>
-    <xacro:link_with_sc no_prefix="${no_prefix}" name="link0" gazebo="${gazebo}" with_sc="${with_sc}">
+    <xacro:link_with_sc no_prefix="${no_prefix}" name="link0" gazebo="${gazebo}" with_sc="${with_sc}" mesh_model="${mesh_model}">
       <self_collision_geometries>
         <xacro:collision_capsule xyz="-0.075 0 0.06" direction="x" radius="${0.06+safety_distance}" length="0.03" />
       </self_collision_geometries>
     </xacro:link_with_sc>
-    <xacro:link_with_sc no_prefix="${no_prefix}" name="link1" gazebo="${gazebo}" with_sc="${with_sc}">
+    <xacro:link_with_sc no_prefix="${no_prefix}" name="link1" gazebo="${gazebo}" with_sc="${with_sc}" mesh_model="${mesh_model}">
       <self_collision_geometries>
         <xacro:collision_capsule xyz="0 0 -191.5e-3" radius="${0.06+safety_distance}" length="0.283" />
@@ -35,5 +35,5 @@
       <xacro:franka-dynamics name="joint1" config="${dynamics}" />
     </joint>
-    <xacro:link_with_sc no_prefix="${no_prefix}" name="link2" gazebo="${gazebo}" with_sc="${with_sc}">
+    <xacro:link_with_sc no_prefix="${no_prefix}" name="link2" gazebo="${gazebo}" with_sc="${with_sc}" mesh_model="${mesh_model}">
       <self_collision_geometries>
         <xacro:collision_capsule xyz="0 0 0" radius="${0.06+safety_distance}" length="0.12" />
@@ -48,5 +48,5 @@
       <xacro:franka-dynamics name="joint2" config="${dynamics}" />
     </joint>
-    <xacro:link_with_sc no_prefix="${no_prefix}" name="link3" gazebo="${gazebo}" with_sc="${with_sc}">
+    <xacro:link_with_sc no_prefix="${no_prefix}" name="link3" gazebo="${gazebo}" with_sc="${with_sc}" mesh_model="${mesh_model}">
       <self_collision_geometries>
         <xacro:collision_capsule xyz="0 0 -0.145" radius="${0.06+safety_distance}" length="0.15" />
@@ -61,5 +61,5 @@
       <xacro:franka-dynamics name="joint3" config="${dynamics}" />
     </joint>
-    <xacro:link_with_sc no_prefix="${no_prefix}" name="link4" gazebo="${gazebo}" with_sc="${with_sc}">
+    <xacro:link_with_sc no_prefix="${no_prefix}" name="link4" gazebo="${gazebo}" with_sc="${with_sc}" mesh_model="${mesh_model}">
       <self_collision_geometries>
         <xacro:collision_capsule xyz="0 0 0" radius="${0.06+safety_distance}" length="0.12" />
@@ -74,5 +74,5 @@
       <xacro:franka-dynamics name="joint4" config="${dynamics}" />
     </joint>
-    <xacro:link_with_sc no_prefix="${no_prefix}" name="link5" gazebo="${gazebo}" with_sc="${with_sc}">
+    <xacro:link_with_sc no_prefix="${no_prefix}" name="link5" gazebo="${gazebo}" with_sc="${with_sc}" mesh_model="${mesh_model}">
       <self_collision_geometries>
         <xacro:collision_capsule xyz="0 0 -0.26"    radius="${0.060+safety_distance}" length="0.10" />
@@ -88,5 +88,5 @@
       <xacro:franka-dynamics name="joint5" config="${dynamics}" />
     </joint>
-    <xacro:link_with_sc no_prefix="${no_prefix}" name="link6" gazebo="${gazebo}" with_sc="${with_sc}">
+    <xacro:link_with_sc no_prefix="${no_prefix}" name="link6" gazebo="${gazebo}" with_sc="${with_sc}" mesh_model="${mesh_model}">
       <self_collision_geometries>
         <xacro:collision_capsule xyz="0 0 -0.03" radius="${0.05+safety_distance}" length="0.08" />
@@ -101,5 +101,5 @@
       <xacro:franka-dynamics name="joint6" config="${dynamics}" />
     </joint>
-    <xacro:link_with_sc no_prefix="${no_prefix}" name="link7" gazebo="${gazebo}" rpy="0 0 ${pi/4}" with_sc="${with_sc}">
+    <xacro:link_with_sc no_prefix="${no_prefix}" name="link7" gazebo="${gazebo}" rpy="0 0 ${pi/4}" with_sc="${with_sc}" mesh_model="${mesh_model}">
       <self_collision_geometries>
         <xacro:collision_capsule xyz="0 0 0.01" direction="z" radius="${0.04+safety_distance}" length="0.14" />

File: robots/common/franka_robot.xacro (robot description, xacro)
@@ -29,5 +29,7 @@
                       description_pkg:='franka_description'
                       connected_to:='base'
-                      scheduling_policy:='detached'">
+                      scheduling_policy:='detached'
+                      mesh_model:=''
+                      ">
     <xacro:include filename="$(find franka_description)/robots/common/utils.xacro" />
     <xacro:include filename="$(find franka_description)/robots/common/franka_arm.xacro" />
@@ -46,4 +48,5 @@
       with_sc="${with_sc}"
       connected_to="${connected_to}"
+      mesh_model="${mesh_model}"
     />
     <xacro:if value="${hand and ee_id == 'franka_hand'}">

File: robots/common/utils.xacro (robot description, xacro)
@@ -32,16 +32,17 @@
   <!-- self_collision_geometries:  self <collision> models        -->
   <!-- ========================================================== -->
-  <xacro:macro name="link_with_sc" params="name no_prefix:='false' rpy:='0 0 0' **self_collision_geometries gazebo:=false with_sc:=false">
+  <xacro:macro name="link_with_sc" params="name no_prefix:='false' rpy:='0 0 0' **self_collision_geometries gazebo:=false with_sc:=false mesh_model:=''">
     <xacro:property name="prefix" value="${'' if no_prefix else arm_prefix + arm_id + '_'}" />
+    <xacro:property name="mesh_id" value="${mesh_model if mesh_model else arm_id}" />
     <!-- sub-link defining detailed meshes for collision with environment -->
     <link name="${prefix}${name}">
       <visual name="${prefix}${name}_visual">
         <geometry>
-          <mesh filename="package://${description_pkg}/meshes/robot_arms/${arm_id}/visual/${name}.dae" />
+          <mesh filename="package://${description_pkg}/meshes/robot_arms/${mesh_id}/visual/${name}.dae" />
         </geometry>
       </visual>
       <collision name="${prefix}${name}_collision">
         <geometry>
-          <mesh filename="package://franka_description/meshes/robot_arms/${arm_id}/collision/${name}.stl" />
+          <mesh filename="package://franka_description/meshes/robot_arms/${mesh_id}/collision/${name}.stl" />
         </geometry>
       </collision>

Commit message: Define velocity, pose and elbow command interfaces when using real or isaac sim hardware

File: robots/common/franka_arm.ros2_control.xacro (robot description, xacro)
@@ -35,6 +35,7 @@
           <xacro:if value="${ros2_control_hardware_type == 'isaac' and gazebo == 0}">
             <plugin>topic_based_ros2_control/TopicBasedSystem</plugin>
-            <param name="joint_commands_topic">/isaac_joint_commands</param>
-            <param name="joint_states_topic">/isaac_joint_states</param>
+            <param name="joint_commands_topic">/isaac/command/left_robot</param>
+            <param name="joint_commands_topic">/isaac/command/right_robot</param>
+            <param name="joint_states_topic">/isaac/joint_states</param>
           </xacro:if>
           <!--- Real Hardware -->
@@ -83,22 +84,25 @@
         </gpio>
       </xacro:macro>
-      <!-- Cartesian velocity interfaces -->
-      <xacro:general_purpose_io prefix="${arm_prefix_modified}vx" command_interface="cartesian_velocity" index="0"/>
-      <xacro:general_purpose_io prefix="${arm_prefix_modified}vy" command_interface="cartesian_velocity" index="1"/>
-      <xacro:general_purpose_io prefix="${arm_prefix_modified}vz" command_interface="cartesian_velocity" index="2"/>
-      <xacro:general_purpose_io prefix="${arm_prefix_modified}wx" command_interface="cartesian_velocity" index="3"/>
-      <xacro:general_purpose_io prefix="${arm_prefix_modified}wy" command_interface="cartesian_velocity" index="4"/>
-      <xacro:general_purpose_io prefix="${arm_prefix_modified}wz" command_interface="cartesian_velocity" index="5"/>
-      <!-- Cartesian pose interfaces, in total 16 interfaces -->
-      <xacro:macro name="loop" params="i">
-        <xacro:unless value="${i == 16}">
-          <xacro:general_purpose_io prefix="${arm_prefix_modified}${i}" command_interface="cartesian_pose_command" index="${i}"/>
-          <xacro:loop i="${i+1}"/>
-        </xacro:unless>
-      </xacro:macro>
-      <xacro:loop i="0"/>
-      <!-- Elbow command interfaces -->
-      <xacro:general_purpose_io prefix="${arm_prefix_modified}joint_3_position" command_interface="elbow_command" index="0"/>
-      <xacro:general_purpose_io prefix="${arm_prefix_modified}joint_4_sign" command_interface="elbow_command" index="1"/>
+      <!-- Franka-specific GPIO interfaces: not supported by mock_components/GenericSystem -->
+      <xacro:if value="${ros2_control_hardware_type == 'real' or ros2_control_hardware_type == 'isaac'}">
+        <!-- Cartesian velocity interfaces -->
+        <xacro:general_purpose_io prefix="${arm_prefix_modified}vx" command_interface="cartesian_velocity" index="0"/>
+        <xacro:general_purpose_io prefix="${arm_prefix_modified}vy" command_interface="cartesian_velocity" index="1"/>
+        <xacro:general_purpose_io prefix="${arm_prefix_modified}vz" command_interface="cartesian_velocity" index="2"/>
+        <xacro:general_purpose_io prefix="${arm_prefix_modified}wx" command_interface="cartesian_velocity" index="3"/>
+        <xacro:general_purpose_io prefix="${arm_prefix_modified}wy" command_interface="cartesian_velocity" index="4"/>
+        <xacro:general_purpose_io prefix="${arm_prefix_modified}wz" command_interface="cartesian_velocity" index="5"/>
+        <!-- Cartesian pose interfaces, in total 16 interfaces -->
+        <xacro:macro name="loop" params="i">
+          <xacro:unless value="${i == 16}">
+            <xacro:general_purpose_io prefix="${arm_prefix_modified}${i}" command_interface="cartesian_pose_command" index="${i}"/>
+            <xacro:loop i="${i+1}"/>
+          </xacro:unless>
+        </xacro:macro>
+        <xacro:loop i="0"/>
+        <!-- Elbow command interfaces -->
+        <xacro:general_purpose_io prefix="${arm_prefix_modified}joint_3_position" command_interface="elbow_command" index="0"/>
+        <xacro:general_purpose_io prefix="${arm_prefix_modified}joint_4_sign" command_interface="elbow_command" index="1"/>
+      </xacro:if>
     </ros2_control>
     <xacro:if value="${gazebo}">
