Commit message: update description for the manipualtion scenario

File: end_effectors/franka_hand/franka_hand.srdf.xacro (robot description, xacro)
@@ -4,4 +4,6 @@
     <group name="${prefix}hand">
       <link name="${prefix}hand"/>
+      <link name="${prefix}hand_tcp"/>
+      <link name="finger_tip_tcp"/>
       <link name="${prefix}leftfinger"/>
       <link name="${prefix}rightfinger"/>

File: robots/fr3/fr3.urdf.xacro (robot description, xacro)
@@ -48,4 +48,5 @@
     </joint>
   </xacro:if>
+  <link name="base" />
   <xacro:franka_robot robot_type="fr3"
     gazebo="$(arg gazebo)"

Commit message: update description for the manipualtion scenario

File: end_effectors/franka_hand/franka_hand.srdf.xacro (robot description, xacro)
@@ -4,4 +4,6 @@
     <group name="${prefix}hand">
       <link name="${prefix}hand"/>
+      <link name="${prefix}hand_tcp"/>
+      <link name="finger_tip_tcp"/>
       <link name="${prefix}leftfinger"/>
       <link name="${prefix}rightfinger"/>

File: robots/fr3/fr3.urdf.xacro (robot description, xacro)
@@ -47,4 +47,5 @@
   <xacro:property name="prefix" value="$(arg arm_prefix)"/>
   <xacro:property name="modified_prefix" value="${prefix + '_' if prefix else ''}"/>
+  <link name="base" />
   <xacro:franka_robot arm_id="fr3"
                       joint_limits="${xacro.load_yaml('$(find franka_description)/robots/fr3/joint_limits.yaml')}"
