Commit message: update description for the manipualtion scenario

File: robots/fr3/fr3.urdf.xacro (robot description, xacro)
@@ -56,4 +56,5 @@
     </joint>
   </xacro:if>
+  <link name="base" />
   <xacro:franka_robot robot_type="fr3"
                       joint_limits="${xacro.load_yaml('$(find franka_description)/robots/fr3/joint_limits.yaml')}"
