Commit message: Remove the arm ID from the prefix

File: end_effectors/common/ee_with_one_link.xacro (robot description, xacro)
@@ -5,5 +5,5 @@
     <xacro:property name="ee_prefix" default="robot_"/>
     <xacro:unless value="${robot_type == ''}">
-      <xacro:property name="ee_prefix" value="${arm_prefix}${robot_type}_" />
+      <xacro:property name="ee_prefix" value="${arm_prefix}" />
     </xacro:unless>
     <xacro:unless value="${connected_to == ''}">

File: end_effectors/common/franka_hand.xacro (robot description, xacro)
@@ -17,5 +17,5 @@
     <xacro:property name="ee_prefix" default="robot_"/>
     <xacro:unless value="${robot_type == ''}">
-      <xacro:property name="ee_prefix" value="${arm_prefix}${robot_type}_" />
+      <xacro:property name="ee_prefix" value="${arm_prefix}" />
     </xacro:unless>
     <xacro:unless value="${connected_to == ''}">

File: robots/common/franka_arm.ros2_control.xacro (robot description, xacro)
@@ -21,5 +21,5 @@
           <param name="version">0.1.0</param>
           <param name="arm_id">${arm_id}</param>
-          <param name="prefix">${arm_prefix}</param>
+          <param name="prefix">${arm_prefix_modified}</param>
           <xacro:if value="${use_fake_hardware}">
             <plugin>mock_components/GenericSystem</plugin>
@@ -33,5 +33,5 @@
             <plugin>franka_hardware/FrankaHardwareInterface</plugin>
             <param name="robot_ip">${robot_ip}</param>
-            <param name="arm_prefix">${arm_prefix}</param>
+            <param name="arm_prefix">${arm_prefix_modified}</param>
           </xacro:if>
         </hardware>
@@ -57,13 +57,13 @@
         </joint>
       </xacro:macro>
-      <xacro:configure_joint joint_name="${arm_prefix}${arm_id}_joint1" initial_position="0.0"/>
-      <xacro:configure_joint joint_name="${arm_prefix}${arm_id}_joint2" initial_position="${-pi/4}"/>
-      <xacro:configure_joint joint_name="${arm_prefix}${arm_id}_joint3" initial_position="0.0"/>
-      <xacro:configure_joint joint_name="${arm_prefix}${arm_id}_joint4" initial_position="${-3*pi/4}"/>
-      <xacro:configure_joint joint_name="${arm_prefix}${arm_id}_joint5" initial_position="0.0"/>
-      <xacro:configure_joint joint_name="${arm_prefix}${arm_id}_joint6" initial_position="${pi/2}"/>
-      <xacro:configure_joint joint_name="${arm_prefix}${arm_id}_joint7" initial_position="${pi/4}"/>
+      <xacro:configure_joint joint_name="${arm_prefix_modified}joint1" initial_position="0.0"/>
+      <xacro:configure_joint joint_name="${arm_prefix_modified}joint2" initial_position="${-pi/4}"/>
+      <xacro:configure_joint joint_name="${arm_prefix_modified}joint3" initial_position="0.0"/>
+      <xacro:configure_joint joint_name="${arm_prefix_modified}joint4" initial_position="${-3*pi/4}"/>
+      <xacro:configure_joint joint_name="${arm_prefix_modified}joint5" initial_position="0.0"/>
+      <xacro:configure_joint joint_name="${arm_prefix_modified}joint6" initial_position="${pi/2}"/>
+      <xacro:configure_joint joint_name="${arm_prefix_modified}joint7" initial_position="${pi/4}"/>
       <xacro:if value="${hand and use_fake_hardware}">
-        <xacro:configure_joint joint_name="${arm_prefix}${arm_id}_finger_joint1" initial_position="0.0" />
+        <xacro:configure_joint joint_name="${arm_prefix_modified}finger_joint1" initial_position="0.0" />
       </xacro:if>
       <xacro:macro name="general_purpose_io" params="prefix command_interface index">
@@ -74,14 +74,14 @@
       </xacro:macro>
       <!-- Cartesian velocity interfaces -->
-      <xacro:general_purpose_io prefix="${arm_prefix}${arm_id}_vx" command_interface="cartesian_velocity" index="0"/>
-      <xacro:general_purpose_io prefix="${arm_prefix}${arm_id}_vy" command_interface="cartesian_velocity" index="1"/>
-      <xacro:general_purpose_io prefix="${arm_prefix}${arm_id}_vz" command_interface="cartesian_velocity" index="2"/>
-      <xacro:general_purpose_io prefix="${arm_prefix}${arm_id}_wx" command_interface="cartesian_velocity" index="3"/>
-      <xacro:general_purpose_io prefix="${arm_prefix}${arm_id}_wy" command_interface="cartesian_velocity" index="4"/>
-      <xacro:general_purpose_io prefix="${arm_prefix}${arm_id}_wz" command_interface="cartesian_velocity" index="5"/>
+      <xacro:general_purpose_io prefix="${arm_prefix_modified}vx" command_interface="cartesian_velocity" index="0"/>
+      <xacro:general_purpose_io prefix="${arm_prefix_modified}vy" command_interface="cartesian_velocity" index="1"/>
+      <xacro:general_purpose_io prefix="${arm_prefix_modified}vz" command_interface="cartesian_velocity" index="2"/>
+      <xacro:general_purpose_io prefix="${arm_prefix_modified}wx" command_interface="cartesian_velocity" index="3"/>
+      <xacro:general_purpose_io prefix="${arm_prefix_modified}wy" command_interface="cartesian_velocity" index="4"/>
+      <xacro:general_purpose_io prefix="${arm_prefix_modified}wz" command_interface="cartesian_velocity" index="5"/>
       <!-- Cartesian pose interfaces, in total 16 interfaces -->
       <xacro:macro name="loop" params="i">
         <xacro:unless value="${i == 16}">
-          <xacro:general_purpose_io prefix="${arm_prefix}${arm_id}_${i}" command_interface="cartesian_pose_command" index="${i}"/>
+          <xacro:general_purpose_io prefix="${arm_prefix_modified}${i}" command_interface="cartesian_pose_command" index="${i}"/>
           <xacro:loop i="${i+1}"/>
         </xacro:unless>
@@ -89,6 +89,6 @@
       <xacro:loop i="0"/>
       <!-- Elbow command interfaces -->
-      <xacro:general_purpose_io prefix="${arm_prefix}${arm_id}_joint_3_position" command_interface="elbow_command" index="0"/>
-      <xacro:general_purpose_io prefix="${arm_prefix}${arm_id}_joint_4_sign" command_interface="elbow_command" index="1"/>
+      <xacro:general_purpose_io prefix="${arm_prefix_modified}joint_3_position" command_interface="elbow_command" index="0"/>
+      <xacro:general_purpose_io prefix="${arm_prefix_modified}joint_4_sign" command_interface="elbow_command" index="1"/>
     </ros2_control>
     <xacro:if value="${gazebo}">

File: robots/common/franka_arm.srdf.xacro (robot description, xacro)
@@ -2,5 +2,5 @@
 <robot xmlns:xacro="http://www.ros.org/wiki/xacro" >
     <xacro:macro name="franka_arm_srdf" params="robot_type hand:='true' ee_id:=franka_hand arm_prefix='' no_prefix='false'">
-        <xacro:property name="prefix" value="${'' if no_prefix else arm_prefix + robot_type + '_'}" />
+        <xacro:property name="prefix" value="${'' if no_prefix else arm_prefix + '_'}" />
         <xacro:include filename="$(find franka_description)/robots/common/group_definition.xacro"/>
         <xacro:property name="tip_link" value="${prefix + 'hand_tcp' if hand and ee_id == 'franka_hand' else prefix + 'link8'}"/>

File: robots/common/franka_arm.xacro (robot description, xacro)
@@ -15,5 +15,5 @@
     <xacro:property name="dynamics" value="${xacro.load_yaml('$(find franka_description)/robots/' + robot_type + '/dynamics.yaml')}"/>
     <!-- Define a property that defaults to 'arm_prefix_robot_type' concatenated with an underscore if 'no_prefix' is not set -->
-    <xacro:property name="prefix" value="${'' if no_prefix else arm_prefix + robot_type + '_'}" />
+    <xacro:property name="prefix" value="${'' if no_prefix else arm_prefix + '_'}" />
     <xacro:property name="with_accelerometers" value="${'false' if accelerometer_config == 'none' else 'true'}" />
     <xacro:if value="${gazebo and connected_to == 'base'}">

File: robots/common/franka_robot.xacro (robot description, xacro)
@@ -29,4 +29,5 @@
     <xacro:include filename="$(find franka_description)/robots/common/utils.xacro" />
     <xacro:include filename="$(find franka_description)/robots/common/franka_arm.xacro"/>
+    <xacro:property name="prefix" value="${'' if arm_prefix == '' else arm_prefix + '_'}" />
     <xacro:franka_arm
       robot_type="${robot_type}"
@@ -92,59 +93,59 @@
     <!-- Definition of additional Gazebo tags -->
     <xacro:if value="${gazebo}">
-      <xacro:gazebo-joint joint="${arm_prefix}${robot_type}_joint1"
+      <xacro:gazebo-joint joint="${prefix}joint1"
         transmission="hardware_interface/PositionJointInterface"/>
-      <xacro:gazebo-joint joint="${arm_prefix}${robot_type}_joint2"
+      <xacro:gazebo-joint joint="${prefix}joint2"
         transmission="hardware_interface/PositionJointInterface"/>
-      <xacro:gazebo-joint joint="${arm_prefix}${robot_type}_joint3"
+      <xacro:gazebo-joint joint="${prefix}joint3"
         transmission="hardware_interface/PositionJointInterface"/>
-      <xacro:gazebo-joint joint="${arm_prefix}${robot_type}_joint4"
+      <xacro:gazebo-joint joint="${prefix}joint4"
         transmission="hardware_interface/PositionJointInterface"/>
-      <xacro:gazebo-joint joint="${arm_prefix}${robot_type}_joint5"
+      <xacro:gazebo-joint joint="${prefix}joint5"
         transmission="hardware_interface/PositionJointInterface"/>
-      <xacro:gazebo-joint joint="${arm_prefix}${robot_type}_joint6"
+      <xacro:gazebo-joint joint="${prefix}joint6"
         transmission="hardware_interface/PositionJointInterface"/>
-      <xacro:gazebo-joint joint="${arm_prefix}${robot_type}_joint7"
+      <xacro:gazebo-joint joint="${prefix}joint7"
         transmission="hardware_interface/PositionJointInterface"/>
-      <xacro:gazebo-joint joint="${arm_prefix}${robot_type}_joint1"
+      <xacro:gazebo-joint joint="${prefix}joint1"
         transmission="hardware_interface/VelocityJointInterface"/>
-      <xacro:gazebo-joint joint="${arm_prefix}${robot_type}_joint2"
+      <xacro:gazebo-joint joint="${prefix}joint2"
         transmission="hardware_interface/VelocityJointInterface"/>
-      <xacro:gazebo-joint joint="${arm_prefix}${robot_type}_joint3"
+      <xacro:gazebo-joint joint="${prefix}joint3"
         transmission="hardware_interface/VelocityJointInterface"/>
-      <xacro:gazebo-joint joint="${arm_prefix}${robot_type}_joint4"
+      <xacro:gazebo-joint joint="${prefix}joint4"
         transmission="hardware_interface/VelocityJointInterface"/>
-      <xacro:gazebo-joint joint="${arm_prefix}${robot_type}_joint5"
+      <xacro:gazebo-joint joint="${prefix}joint5"
         transmission="hardware_interface/VelocityJointInterface"/>
-      <xacro:gazebo-joint joint="${arm_prefix}${robot_type}_joint6"
+      <xacro:gazebo-joint joint="${prefix}joint6"
         transmission="hardware_interface/VelocityJointInterface"/>
-      <xacro:gazebo-joint joint="${arm_prefix}${robot_type}_joint7"
+      <xacro:gazebo-joint joint="${prefix}joint7"
         transmission="hardware_interface/VelocityJointInterface"/>
-      <xacro:gazebo-joint joint="${arm_prefix}${robot_type}_joint1"
+      <xacro:gazebo-joint joint="${prefix}joint1"
         transmission="hardware_interface/EffortJointInterface"/>
-      <xacro:gazebo-joint joint="${arm_prefix}${robot_type}_joint2"
+      <xacro:gazebo-joint joint="${prefix}joint2"
         transmission="hardware_interface/EffortJointInterface"/>
-      <xacro:gazebo-joint joint="${arm_prefix}${robot_type}_joint3"
+      <xacro:gazebo-joint joint="${prefix}joint3"
         transmission="hardware_interface/EffortJointInterface"/>
-      <xacro:gazebo-joint joint="${arm_prefix}${robot_type}_joint4"
+      <xacro:gazebo-joint joint="${prefix}joint4"
         transmission="hardware_interface/EffortJointInterface"/>
-      <xacro:gazebo-joint joint="${arm_prefix}${robot_type}_joint5"
+      <xacro:gazebo-joint joint="${prefix}joint5"
         transmission="hardware_interface/EffortJointInterface"/>
-      <xacro:gazebo-joint joint="${arm_prefix}${robot_type}_joint6"
+      <xacro:gazebo-joint joint="${prefix}joint6"
         transmission="hardware_interface/EffortJointInterface"/>
-      <xacro:gazebo-joint joint="${arm_prefix}${robot_type}_joint7"
+      <xacro:gazebo-joint joint="${prefix}joint7"
         transmission="hardware_interface/EffortJointInterface"/>
       <xacro:transmission-franka-state robot_type="${robot_type}"/>
       <xacro:transmission-franka-model robot_type="${robot_type}"
-        root="${arm_prefix}${robot_type}_joint1"
-        tip="${arm_prefix}${robot_type}_joint8"
+        root="${prefix}joint1"
+        tip="${prefix}joint8"
       />
       <xacro:if value="${ee_id == 'franka_hand'}">
-        <xacro:gazebo-joint joint="${arm_prefix}${robot_type}_finger_joint1"
+        <xacro:gazebo-joint joint="${prefix}finger_joint1"
           transmission="hardware_interface/EffortJointInterface"/>
-        <xacro:gazebo-joint joint="${arm_prefix}${robot_type}_finger_joint2"
+        <xacro:gazebo-joint joint="${prefix}finger_joint2"
           transmission="hardware_interface/EffortJointInterface"/>
         <!-- Friction specific material for Rubber/Rubber contact -->
-        <xacro:gazebo-friction link="${arm_prefix}${robot_type}_leftfinger" mu="1.13"/>
-        <xacro:gazebo-friction link="${arm_prefix}${robot_type}_rightfinger" mu="1.13"/>
+        <xacro:gazebo-friction link="${prefix}leftfinger" mu="1.13"/>
+        <xacro:gazebo-friction link="${prefix}rightfinger" mu="1.13"/>
       </xacro:if>
     </xacro:if>

File: robots/common/utils.xacro (robot description, xacro)
@@ -33,5 +33,5 @@
   <!-- ========================================================== -->
   <xacro:macro name="link_with_sc" params="name no_prefix:='false' rpy:='0 0 0' **self_collision_geometries gazebo:=false with_sc:=false with_accelerometers:=false mesh_model:=''">
-    <xacro:property name="prefix" value="${'' if no_prefix else arm_prefix + robot_type + '_'}" />
+    <xacro:property name="prefix" value="${'' if no_prefix else arm_prefix + '_'}" />
     <xacro:property name="mesh_id" value="${mesh_model if mesh_model else robot_type}" />
     <!-- sub-link defining detailed meshes for collision with environment -->
@@ -161,20 +161,20 @@
   <!-- ========================================================== -->
   <xacro:macro name="transmission-franka-state" params="robot_type:=fer">
-    <transmission name="${arm_prefix}${robot_type}_franka_state">
+    <transmission name="${arm_prefix}franka_state">
       <type>franka_hw/FrankaStateInterface</type>
-      <joint name="${arm_prefix}${robot_type}_joint1"><hardwareInterface>franka_hw/FrankaStateInterface</hardwareInterface></joint>
-      <joint name="${arm_prefix}${robot_type}_joint2"><hardwareInterface>franka_hw/FrankaStateInterface</hardwareInterface></joint>
-      <joint name="${arm_prefix}${robot_type}_joint3"><hardwareInterface>franka_hw/FrankaStateInterface</hardwareInterface></joint>
-      <joint name="${arm_prefix}${robot_type}_joint4"><hardwareInterface>franka_hw/FrankaStateInterface</hardwareInterface></joint>
-      <joint name="${arm_prefix}${robot_type}_joint5"><hardwareInterface>franka_hw/FrankaStateInterface</hardwareInterface></joint>
-      <joint name="${arm_prefix}${robot_type}_joint6"><hardwareInterface>franka_hw/FrankaStateInterface</hardwareInterface></joint>
-      <joint name="${arm_prefix}${robot_type}_joint7"><hardwareInterface>franka_hw/FrankaStateInterface</hardwareInterface></joint>
-      <actuator name="${arm_prefix}${robot_type}_motor1"><hardwareInterface>franka_hw/FrankaStateInterface</hardwareInterface></actuator>
-      <actuator name="${arm_prefix}${robot_type}_motor2"><hardwareInterface>franka_hw/FrankaStateInterface</hardwareInterface></actuator>
-      <actuator name="${arm_prefix}${robot_type}_motor3"><hardwareInterface>franka_hw/FrankaStateInterface</hardwareInterface></actuator>
-      <actuator name="${arm_prefix}${robot_type}_motor4"><hardwareInterface>franka_hw/FrankaStateInterface</hardwareInterface></actuator>
-      <actuator name="${arm_prefix}${robot_type}_motor5"><hardwareInterface>franka_hw/FrankaStateInterface</hardwareInterface></actuator>
-      <actuator name="${arm_prefix}${robot_type}_motor6"><hardwareInterface>franka_hw/FrankaStateInterface</hardwareInterface></actuator>
-      <actuator name="${arm_prefix}${robot_type}_motor7"><hardwareInterface>franka_hw/FrankaStateInterface</hardwareInterface></actuator>
+      <joint name="${arm_prefix}joint1"><hardwareInterface>franka_hw/FrankaStateInterface</hardwareInterface></joint>
+      <joint name="${arm_prefix}joint2"><hardwareInterface>franka_hw/FrankaStateInterface</hardwareInterface></joint>
+      <joint name="${arm_prefix}joint3"><hardwareInterface>franka_hw/FrankaStateInterface</hardwareInterface></joint>
+      <joint name="${arm_prefix}joint4"><hardwareInterface>franka_hw/FrankaStateInterface</hardwareInterface></joint>
+      <joint name="${arm_prefix}joint5"><hardwareInterface>franka_hw/FrankaStateInterface</hardwareInterface></joint>
+      <joint name="${arm_prefix}joint6"><hardwareInterface>franka_hw/FrankaStateInterface</hardwareInterface></joint>
+      <joint name="${arm_prefix}joint7"><hardwareInterface>franka_hw/FrankaStateInterface</hardwareInterface></joint>
+      <actuator name="${arm_prefix}motor1"><hardwareInterface>franka_hw/FrankaStateInterface</hardwareInterface></actuator>
+      <actuator name="${arm_prefix}motor2"><hardwareInterface>franka_hw/FrankaStateInterface</hardwareInterface></actuator>
+      <actuator name="${arm_prefix}motor3"><hardwareInterface>franka_hw/FrankaStateInterface</hardwareInterface></actuator>
+      <actuator name="${arm_prefix}motor4"><hardwareInterface>franka_hw/FrankaStateInterface</hardwareInterface></actuator>
+      <actuator name="${arm_prefix}motor5"><hardwareInterface>franka_hw/FrankaStateInterface</hardwareInterface></actuator>
+      <actuator name="${arm_prefix}motor6"><hardwareInterface>franka_hw/FrankaStateInterface</hardwareInterface></actuator>
+      <actuator name="${arm_prefix}motor7"><hardwareInterface>franka_hw/FrankaStateInterface</hardwareInterface></actuator>
     </transmission>
   </xacro:macro>
@@ -188,5 +188,5 @@
   <!-- ============================================================ -->
   <xacro:macro name="transmission-franka-model" params="robot_type:=fer root:=fer_joint1 tip:=fer_joint7">
-    <transmission name="${arm_prefix}${robot_type}_franka_model">
+    <transmission name="${arm_prefix}franka_model">
       <type>franka_hw/FrankaModelInterface</type>
       <joint name="${root}">
