Commit message: Remove the arm ID from the prefix

File: end_effectors/common/ee_with_one_link.xacro (robot description, xacro)
@@ -5,5 +5,5 @@
     <xacro:property name="ee_prefix" default="robot_"/>
     <xacro:unless value="${robot_type == ''}">
-      <xacro:property name="ee_prefix" value="${arm_prefix}${robot_type}_" />
+      <xacro:property name="ee_prefix" value="${arm_prefix}" />
     </xacro:unless>
     <xacro:unless value="${connected_to == ''}">

File: end_effectors/common/franka_hand.xacro (robot description, xacro)
@@ -17,5 +17,5 @@
     <xacro:property name="ee_prefix" default="robot_"/>
     <xacro:unless value="${robot_type == ''}">
-      <xacro:property name="ee_prefix" value="${arm_prefix}${robot_type}_" />
+      <xacro:property name="ee_prefix" value="${arm_prefix}" />
     </xacro:unless>
     <xacro:unless value="${connected_to == ''}">

File: robots/common/franka_arm.ros2_control.xacro (robot description, xacro)
@@ -23,5 +23,5 @@
           <param name="version">1.0.0</param>
           <param name="robot_type">${robot_type}</param>
-          <param name="prefix">${arm_prefix}</param>
+          <param name="prefix">${arm_prefix_modified}</param>
           <xacro:if value="${use_fake_hardware}">
             <plugin>mock_components/GenericSystem</plugin>
@@ -35,5 +35,5 @@
             <plugin>franka_hardware/FrankaHardwareInterface</plugin>
             <param name="robot_ip">${robot_ip}</param>
-            <param name="arm_prefix">${arm_prefix}</param>
+            <param name="arm_prefix">${arm_prefix_modified}</param>
           </xacro:if>
         </hardware>
@@ -59,13 +59,13 @@
         </joint>
       </xacro:macro>
-      <xacro:configure_joint joint_name="${arm_prefix}${robot_type}_joint1" initial_position="0.0"/>
-      <xacro:configure_joint joint_name="${arm_prefix}${robot_type}_joint2" initial_position="${-pi/4}"/>
-      <xacro:configure_joint joint_name="${arm_prefix}${robot_type}_joint3" initial_position="0.0"/>
-      <xacro:configure_joint joint_name="${arm_prefix}${robot_type}_joint4" initial_position="${-3*pi/4}"/>
-      <xacro:configure_joint joint_name="${arm_prefix}${robot_type}_joint5" initial_position="0.0"/>
-      <xacro:configure_joint joint_name="${arm_prefix}${robot_type}_joint6" initial_position="${pi/2}"/>
-      <xacro:configure_joint joint_name="${arm_prefix}${robot_type}_joint7" initial_position="${pi/4}"/>
+      <xacro:configure_joint joint_name="${arm_prefix_modified}joint1" initial_position="0.0"/>
+      <xacro:configure_joint joint_name="${arm_prefix_modified}joint2" initial_position="${-pi/4}"/>
+      <xacro:configure_joint joint_name="${arm_prefix_modified}joint3" initial_position="0.0"/>
+      <xacro:configure_joint joint_name="${arm_prefix_modified}joint4" initial_position="${-3*pi/4}"/>
+      <xacro:configure_joint joint_name="${arm_prefix_modified}joint5" initial_position="0.0"/>
+      <xacro:configure_joint joint_name="${arm_prefix_modified}joint6" initial_position="${pi/2}"/>
+      <xacro:configure_joint joint_name="${arm_prefix_modified}joint7" initial_position="${pi/4}"/>
       <xacro:if value="${gazebo and hand}">
-        <xacro:configure_joint joint_name="${arm_prefix}${robot_type}_finger_joint1" initial_position="0.0" />
+        <xacro:configure_joint joint_name="${arm_prefix_modified}finger_joint1" initial_position="0.0" />
       </xacro:if>
       <xacro:macro name="general_purpose_io" params="prefix command_interface index">
@@ -76,14 +76,14 @@
       </xacro:macro>
       <!-- Cartesian velocity interfaces -->
-      <xacro:general_purpose_io prefix="${arm_prefix}${arm_id}_vx" command_interface="cartesian_velocity" index="0"/>
-      <xacro:general_purpose_io prefix="${arm_prefix}${arm_id}_vy" command_interface="cartesian_velocity" index="1"/>
-      <xacro:general_purpose_io prefix="${arm_prefix}${arm_id}_vz" command_interface="cartesian_velocity" index="2"/>
-      <xacro:general_purpose_io prefix="${arm_prefix}${arm_id}_wx" command_interface="cartesian_velocity" index="3"/>
-      <xacro:general_purpose_io prefix="${arm_prefix}${arm_id}_wy" command_interface="cartesian_velocity" index="4"/>
-      <xacro:general_purpose_io prefix="${arm_prefix}${arm_id}_wz" command_interface="cartesian_velocity" index="5"/>
+      <xacro:general_purpose_io prefix="${arm_prefix_modified}vx" command_interface="cartesian_velocity" index="0"/>
+      <xacro:general_purpose_io prefix="${arm_prefix_modified}vy" command_interface="cartesian_velocity" index="1"/>
+      <xacro:general_purpose_io prefix="${arm_prefix_modified}vz" command_interface="cartesian_velocity" index="2"/>
+      <xacro:general_purpose_io prefix="${arm_prefix_modified}wx" command_interface="cartesian_velocity" index="3"/>
+      <xacro:general_purpose_io prefix="${arm_prefix_modified}wy" command_interface="cartesian_velocity" index="4"/>
+      <xacro:general_purpose_io prefix="${arm_prefix_modified}wz" command_interface="cartesian_velocity" index="5"/>
       <!-- Cartesian pose interfaces, in total 16 interfaces -->
       <xacro:macro name="loop" params="i">
         <xacro:unless value="${i == 16}">
-          <xacro:general_purpose_io prefix="${arm_prefix}${arm_id}_${i}" command_interface="cartesian_pose_command" index="${i}"/>
+          <xacro:general_purpose_io prefix="${arm_prefix_modified}${i}" command_interface="cartesian_pose_command" index="${i}"/>
           <xacro:loop i="${i+1}"/>
         </xacro:unless>
@@ -91,6 +91,6 @@
       <xacro:loop i="0"/>
       <!-- Elbow command interfaces -->
-      <xacro:general_purpose_io prefix="${arm_prefix}${arm_id}_joint_3_position" command_interface="elbow_command" index="0"/>
-      <xacro:general_purpose_io prefix="${arm_prefix}${arm_id}_joint_4_sign" command_interface="elbow_command" index="1"/>
+      <xacro:general_purpose_io prefix="${arm_prefix_modified}joint_3_position" command_interface="elbow_command" index="0"/>
+      <xacro:general_purpose_io prefix="${arm_prefix_modified}joint_4_sign" command_interface="elbow_command" index="1"/>
     </ros2_control>
     <xacro:if value="${gazebo}">

File: robots/common/franka_arm.xacro (robot description, xacro)
@@ -10,5 +10,5 @@
   <xacro:macro name="franka_arm" params="robot_type arm_prefix:='' no_prefix:=false description_pkg:='franka_description' connected_to:='base' xyz:='0 0 0' rpy:='0 0 0' gazebo:='false' safety_distance:=0 joint_limits inertials kinematics accelerometer_config dynamics with_sc:=false mesh_model:=''" >
     <!-- Define a property that defaults to 'arm_prefix_robot_type' concatenated with an underscore if 'no_prefix' is not set -->
-    <xacro:property name="prefix" value="${'' if no_prefix else arm_prefix + robot_type + '_'}" />
+    <xacro:property name="prefix" value="${'' if no_prefix else arm_prefix + '_'}" />
     <xacro:property name="with_accelerometers" value="${'false' if accelerometer_config == 'none' else 'true'}" />
     <xacro:if value="${gazebo and connected_to == 'base'}">

File: robots/common/franka_robot.xacro (robot description, xacro)
@@ -36,4 +36,5 @@
     <xacro:include filename="$(find franka_description)/robots/common/utils.xacro" />
     <xacro:include filename="$(find franka_description)/robots/common/franka_arm.xacro"/>
+    <xacro:property name="prefix" value="${'' if arm_prefix == '' else arm_prefix + '_'}" />
     <xacro:franka_arm
       robot_type="${robot_type}"
@@ -101,36 +102,36 @@
     <!-- Definition of additional Gazebo tags -->
     <xacro:if value="${gazebo}">
-      <xacro:gazebo-joint joint="${arm_prefix}${robot_type}_joint1" transmission="hardware_interface/PositionJointInterface" />
-      <xacro:gazebo-joint joint="${arm_prefix}${robot_type}_joint2" transmission="hardware_interface/PositionJointInterface" />
-      <xacro:gazebo-joint joint="${arm_prefix}${robot_type}_joint3" transmission="hardware_interface/PositionJointInterface" />
-      <xacro:gazebo-joint joint="${arm_prefix}${robot_type}_joint4" transmission="hardware_interface/PositionJointInterface" />
-      <xacro:gazebo-joint joint="${arm_prefix}${robot_type}_joint5" transmission="hardware_interface/PositionJointInterface" />
-      <xacro:gazebo-joint joint="${arm_prefix}${robot_type}_joint6" transmission="hardware_interface/PositionJointInterface" />
-      <xacro:gazebo-joint joint="${arm_prefix}${robot_type}_joint7" transmission="hardware_interface/PositionJointInterface" />
-      <xacro:gazebo-joint joint="${arm_prefix}${robot_type}_joint1" transmission="hardware_interface/VelocityJointInterface" />
-      <xacro:gazebo-joint joint="${arm_prefix}${robot_type}_joint2" transmission="hardware_interface/VelocityJointInterface" />
-      <xacro:gazebo-joint joint="${arm_prefix}${robot_type}_joint3" transmission="hardware_interface/VelocityJointInterface" />
-      <xacro:gazebo-joint joint="${arm_prefix}${robot_type}_joint4" transmission="hardware_interface/VelocityJointInterface" />
-      <xacro:gazebo-joint joint="${arm_prefix}${robot_type}_joint5" transmission="hardware_interface/VelocityJointInterface" />
-      <xacro:gazebo-joint joint="${arm_prefix}${robot_type}_joint6" transmission="hardware_interface/VelocityJointInterface" />
-      <xacro:gazebo-joint joint="${arm_prefix}${robot_type}_joint7" transmission="hardware_interface/VelocityJointInterface" />
-      <xacro:gazebo-joint joint="${arm_prefix}${robot_type}_joint1" transmission="hardware_interface/EffortJointInterface" />
-      <xacro:gazebo-joint joint="${arm_prefix}${robot_type}_joint2" transmission="hardware_interface/EffortJointInterface" />
-      <xacro:gazebo-joint joint="${arm_prefix}${robot_type}_joint3" transmission="hardware_interface/EffortJointInterface" />
-      <xacro:gazebo-joint joint="${arm_prefix}${robot_type}_joint4" transmission="hardware_interface/EffortJointInterface" />
-      <xacro:gazebo-joint joint="${arm_prefix}${robot_type}_joint5" transmission="hardware_interface/EffortJointInterface" />
-      <xacro:gazebo-joint joint="${arm_prefix}${robot_type}_joint6" transmission="hardware_interface/EffortJointInterface" />
-      <xacro:gazebo-joint joint="${arm_prefix}${robot_type}_joint7" transmission="hardware_interface/EffortJointInterface" />
+      <xacro:gazebo-joint joint="${prefix}joint1" transmission="hardware_interface/PositionJointInterface" />
+      <xacro:gazebo-joint joint="${prefix}joint2" transmission="hardware_interface/PositionJointInterface" />
+      <xacro:gazebo-joint joint="${prefix}joint3" transmission="hardware_interface/PositionJointInterface" />
+      <xacro:gazebo-joint joint="${prefix}joint4" transmission="hardware_interface/PositionJointInterface" />
+      <xacro:gazebo-joint joint="${prefix}joint5" transmission="hardware_interface/PositionJointInterface" />
+      <xacro:gazebo-joint joint="${prefix}joint6" transmission="hardware_interface/PositionJointInterface" />
+      <xacro:gazebo-joint joint="${prefix}joint7" transmission="hardware_interface/PositionJointInterface" />
+      <xacro:gazebo-joint joint="${prefix}joint1" transmission="hardware_interface/VelocityJointInterface" />
+      <xacro:gazebo-joint joint="${prefix}joint2" transmission="hardware_interface/VelocityJointInterface" />
+      <xacro:gazebo-joint joint="${prefix}joint3" transmission="hardware_interface/VelocityJointInterface" />
+      <xacro:gazebo-joint joint="${prefix}joint4" transmission="hardware_interface/VelocityJointInterface" />
+      <xacro:gazebo-joint joint="${prefix}joint5" transmission="hardware_interface/VelocityJointInterface" />
+      <xacro:gazebo-joint joint="${prefix}joint6" transmission="hardware_interface/VelocityJointInterface" />
+      <xacro:gazebo-joint joint="${prefix}joint7" transmission="hardware_interface/VelocityJointInterface" />
+      <xacro:gazebo-joint joint="${prefix}joint1" transmission="hardware_interface/EffortJointInterface" />
+      <xacro:gazebo-joint joint="${prefix}joint2" transmission="hardware_interface/EffortJointInterface" />
+      <xacro:gazebo-joint joint="${prefix}joint3" transmission="hardware_interface/EffortJointInterface" />
+      <xacro:gazebo-joint joint="${prefix}joint4" transmission="hardware_interface/EffortJointInterface" />
+      <xacro:gazebo-joint joint="${prefix}joint5" transmission="hardware_interface/EffortJointInterface" />
+      <xacro:gazebo-joint joint="${prefix}joint6" transmission="hardware_interface/EffortJointInterface" />
+      <xacro:gazebo-joint joint="${prefix}joint7" transmission="hardware_interface/EffortJointInterface" />
       <xacro:transmission-franka-state robot_type="${robot_type}" />
       <xacro:transmission-franka-model robot_type="${robot_type}"
-         root="${arm_prefix}${robot_type}_joint1"
-         tip="${arm_prefix}${robot_type}_joint8"
+         root="${prefix}joint1"
+         tip="${prefix}joint8"
        />
       <xacro:if value="${ee_id == 'franka_hand'}">
-        <xacro:gazebo-joint joint="${arm_prefix}${robot_type}_finger_joint1" transmission="hardware_interface/EffortJointInterface" />
-        <xacro:gazebo-joint joint="${arm_prefix}${robot_type}_finger_joint2" transmission="hardware_interface/EffortJointInterface" />
+        <xacro:gazebo-joint joint="${prefix}finger_joint1" transmission="hardware_interface/EffortJointInterface" />
+        <xacro:gazebo-joint joint="${prefix}finger_joint2" transmission="hardware_interface/EffortJointInterface" />
         <!-- Friction specific material for Rubber/Rubber contact -->
-        <xacro:gazebo-friction link="${arm_prefix}${robot_type}_leftfinger" mu="1.13" />
-        <xacro:gazebo-friction link="${arm_prefix}${robot_type}_rightfinger" mu="1.13" />
+        <xacro:gazebo-friction link="${prefix}leftfinger" mu="1.13" />
+        <xacro:gazebo-friction link="${prefix}rightfinger" mu="1.13" />
       </xacro:if>
     </xacro:if>
